Commit message: update config files to support third joint motion

File: rrbot_simulation_files/rrbot_description/gazebo/rrbot.gazebo.xacro (robot description, xacro)
@@ -28,4 +28,10 @@
       <material>Gazebo/Orange</material>
     </gazebo>
+    <!-- Link3 -->
+    <gazebo reference="${prefix}link3">
+      <mu1>0.2</mu1>
+      <mu2>0.2</mu2>
+      <material>Gazebo/Red</material>
+    </gazebo>
   </xacro:macro>
 </robot>

File: rrbot_simulation_files/rrbot_description/ros2_control/rrbot.ros2_control.xacro (robot description, xacro)
@@ -46,4 +46,21 @@
         <state_interface name="effort"/>
       </joint>
+      <joint name="${prefix}joint3">
+        <command_interface name="position">
+          <param name="min">-10</param>
+          <param name="max">10</param>
+        </command_interface>
+        <command_interface name="velocity">
+          <param name="min">-10</param>
+          <param name="max">10</param>
+        </command_interface>
+        <command_interface name="effort">
+          <param name="min">-100</param>
+          <param name="max">100</param>
+        </command_interface>
+        <state_interface name="position"/>
+        <state_interface name="velocity"/>
+        <state_interface name="effort"/>
+      </joint>
     </ros2_control>
   </xacro:macro>

File: rrbot_simulation_files/rrbot_description/urdf/rrbot.urdf.xacro (robot description, xacro)
@@ -24,4 +24,4 @@
   <xacro:rrbot_gazebo prefix="$(arg prefix)" />
   <xacro:rrbot_ros2_control
-    name="RRBot" prefix="$(arg prefix)" />
+    name="RRPBot" prefix="$(arg prefix)" />
 </robot>

File: rrbot_simulation_files/rrbot_description/urdf/rrbot_description.urdf.xacro (robot description, xacro)
@@ -100,5 +100,5 @@
         <parent link="link2"/>
         <child link="link3"/>
-        <origin xyz="1 0 ${cyl_height}" rpy="0 0 0"/>
+        <origin xyz="1 0 0" rpy="0 0 0"/>
         <axis xyz="0 0 1"/>
     </joint>
@@ -115,8 +115,7 @@
                 <box size="${l3} ${width} ${width}"/>
            </geometry>
-           <material name="red"/>
         </visual>
         <inertial>
-            <origin xyz="0 0 ${l3/2}" rpy="0 0 0"/>
+            <origin xyz="${l2/2} 0 0" rpy="0 0 0"/>
             <mass value="${mass}"/>
             <inertia
@@ -126,4 +125,35 @@
         </inertial>
     </link>
+    <link name="link4">
+        <collision>
+            <origin xyz="0 0 ${-l4}" rpy="0 0 0"/>
+            <geometry>
+                <box size="0.1 0.1 ${l4}"/>
+            </geometry>
+        </collision>
+        <visual>
+           <origin xyz="${l4} 0 ${-l4}" rpy="0 0 0"/>
+           <geometry>
+                <box size="0.1 0.1 ${l4}"/>
+           </geometry>
+           <material name="red"/>
+        </visual>
+        <inertial>
+            <origin xyz="${l2/2 + l3} 0 0" rpy="0 0 0"/>
+            <mass value="${mass}"/>
+            <inertia
+                ixx="${mass / 12.0 * (width*width + width*width)}" ixy="0.0" ixz="0.0"
+                iyy="${mass / 12.0 * (width*width + l4*l4)}" iyz="0.0"
+                izz="${mass / 12.0 * (width*width + l4*l4)}"/>
+        </inertial>
+    </link>
+    <joint name="joint3" type="prismatic">
+        <parent link="link3"/>
+        <child link="link4"/>
+        <origin xyz="0.0 0.0 ${l4/2}" rpy="0 0 0"/>
+        <axis xyz="0 0 1"/>
+        <limit effort="1000.0" lower="0" upper="1.0" velocity="0.5"/>
+        <dynamics damping="0.7"/>
+    </joint>
   </xacro:macro>
 </robot>
