Commit message: cleaned up comments for submission and removed pseudo variables

File: install/rrbot_description/share/rrbot_description/gazebo/rrbot.gazebo.xacro (robot description, xacro)
@@ -1,37 +1 @@
-<?xml version="1.0"?>
-<!--
-Copied and modified from ROS1 example -
-https://github.com/ros-simulation/gazebo_ros_demos/blob/kinetic-devel/rrbot_description/urdf/rrbot.gazebo
--->
-<robot xmlns:xacro="http://ros.org/wiki/xacro">
-  <xacro:macro name="rrbot_gazebo" params="prefix">
-    <!-- ros_control plugin -->
-    <gazebo>
-      <plugin name="gazebo_ros2_control" filename="libgazebo_ros2_control.so">
-        <parameters>$(find rrbot_gazebo)/config/gazebo_controllers.yaml</parameters>
-      </plugin>
-    </gazebo>
-    <!-- Link1 -->
-    <gazebo reference="${prefix}base_link">
-      <material>Gazebo/Orange</material>
-    </gazebo>
-    <!-- Link2 -->
-    <gazebo reference="${prefix}link1">
-      <mu1>0.2</mu1>
-      <mu2>0.2</mu2>
-      <material>Gazebo/Black</material>
-    </gazebo>
-    <!-- Link3 -->
-    <gazebo reference="${prefix}link2">
-      <mu1>0.2</mu1>
-      <mu2>0.2</mu2>
-      <material>Gazebo/Orange</material>
-    </gazebo>
-    <!-- Link3 -->
-    <gazebo reference="${prefix}link3">
-      <mu1>0.2</mu1>
-      <mu2>0.2</mu2>
-      <material>Gazebo/Red</material>
-    </gazebo>
-  </xacro:macro>
-</robot>
+/home/joshfarina/ros2_ws/src/rbe500_group_project/rrbot_simulation_files/rrbot_description/gazebo/rrbot.gazebo.xacro

File: install/rrbot_description/share/rrbot_description/gazebo/rrbot.materials.xacro (robot description, xacro)
@@ -1,34 +1 @@
-<?xml version="1.0"?>
-<!--
-Copied from ROS1 example -
-https://github.com/ros-simulation/gazebo_ros_demos/blob/kinetic-devel/rrbot_description/urdf/materials.xacro
--->
-<robot>
-  <material name="black">
-    <color rgba="0.0 0.0 0.0 1.0"/>
-  </material>
-  <material name="blue">
-    <color rgba="0.0 0.0 0.8 1.0"/>
-  </material>
-  <material name="green">
-    <color rgba="0.0 0.8 0.0 1.0"/>
-  </material>
-  <material name="grey">
-    <color rgba="0.2 0.2 0.2 1.0"/>
-  </material>
-  <material name="orange">
-    <color rgba="${255/255} ${108/255} ${10/255} 1.0"/>
-  </material>
-  <material name="brown">
-    <color rgba="${222/255} ${207/255} ${195/255} 1.0"/>
-  </material>
-  <material name="red">
-    <color rgba="0.8 0.0 0.0 1.0"/>
-  </material>
-  <material name="yellow">
-    <color rgba="1.0 1.0 0.0 1.0"/>
-  </material>
-  <material name="white">
-    <color rgba="1.0 1.0 1.0 1.0"/>
-  </material>
-</robot>
+/home/joshfarina/ros2_ws/src/rbe500_group_project/rrbot_simulation_files/rrbot_description/gazebo/rrbot.materials.xacro

File: install/rrbot_description/share/rrbot_description/ros2_control/rrbot.ros2_control.xacro (robot description, xacro)
@@ -1,67 +1 @@
-<?xml version="1.0"?>
-<robot xmlns:xacro="http://www.ros.org/wiki/xacro">
-  <xacro:macro name="rrbot_ros2_control" params="name prefix">
-    <ros2_control name="${name}" type="system">
-      <!-- <hardware>
-        <plugin>ros2_control_demo_hardware/RRBotSystemPositionOnlyHardware</plugin>
-        <param name="example_param_hw_start_duration_sec">0</param>
-        <param name="example_param_hw_stop_duration_sec">3.0</param>
-        <param name="example_param_hw_slowdown">100</param>
-      </hardware> -->
-      <hardware>
-          <plugin>gazebo_ros2_control/GazeboSystem</plugin>
-        </hardware>
-      <joint name="${prefix}joint1">
-        <command_interface name="position">
-          <param name="min">-10</param>
-          <param name="max">10</param>
-        </command_interface>
-        <command_interface name="velocity">
-          <param name="min">-10</param>
-          <param name="max">10</param>
-        </command_interface>
-        <command_interface name="effort">
-          <param name="min">-100</param>
-          <param name="max">100</param>
-        </command_interface>
-        <state_interface name="position"/>
-        <state_interface name="velocity"/>
-        <state_interface name="effort"/>
-      </joint>
-      <joint name="${prefix}joint2">
-        <command_interface name="position">
-          <param name="min">-10</param>
-          <param name="max">10</param>
-        </command_interface>
-        <command_interface name="velocity">
-          <param name="min">-10</param>
-          <param name="max">10</param>
-        </command_interface>
-        <command_interface name="effort">
-          <param name="min">-100</param>
-          <param name="max">100</param>
-        </command_interface>
-        <state_interface name="position"/>
-        <state_interface name="velocity"/>
-        <state_interface name="effort"/>
-      </joint>
-      <joint name="${prefix}joint3">
-        <command_interface name="position">
-          <param name="min">-10</param>
-          <param name="max">10</param>
-        </command_interface>
-        <command_interface name="velocity">
-          <param name="min">-10</param>
-          <param name="max">10</param>
-        </command_interface>
-        <command_interface name="effort">
-          <param name="min">-100</param>
-          <param name="max">100</param>
-        </command_interface>
-        <state_interface name="position"/>
-        <state_interface name="velocity"/>
-        <state_interface name="effort"/>
-      </joint>
-    </ros2_control>
-  </xacro:macro>
-</robot>
+/home/joshfarina/ros2_ws/src/rbe500_group_project/rrbot_simulation_files/rrbot_description/ros2_control/rrbot.ros2_control.xacro

File: install/rrbot_description/share/rrbot_description/urdf/rrbot.urdf.xacro (robot description, xacro)
@@ -1,27 +1 @@
-<?xml version="1.0"?>
-<!-- Revolute-Revolute Manipulator -->
-<!--
-Copied and modified from ROS1 example -
-https://github.com/ros-simulation/gazebo_ros_demos/blob/kinetic-devel/rrbot_description/urdf/rrbot.xacro
--->
-<robot xmlns:xacro="http://www.ros.org/wiki/xacro" name="2dof_robot">
-  <xacro:arg name="prefix" default="" />
-  <!-- Import RRBot macro -->
-  <xacro:include filename="$(find rrbot_description)/urdf/rrbot_description.urdf.xacro" />
-  <!-- Import Rviz colors -->
-  <xacro:include filename="$(find rrbot_description)/gazebo/rrbot.materials.xacro" />
-  <!-- Import RRBot ros2_control description -->
-  <xacro:include filename="$(find rrbot_description)/ros2_control/rrbot.ros2_control.xacro" />
-  <xacro:include filename="$(find rrbot_description)/gazebo/rrbot.gazebo.xacro" />
-  <!-- Used for fixing robot -->
-  <link name="world"/>
-  <gazebo reference="world">
-    <static>true</static>
-  </gazebo>
-  <xacro:rrbot parent="world" prefix="$(arg prefix)">
-    <origin xyz="0 0 0" rpy="0 0 0" />
-  </xacro:rrbot>
-  <xacro:rrbot_gazebo prefix="$(arg prefix)" />
-  <xacro:rrbot_ros2_control
-    name="RRPBot" prefix="$(arg prefix)" />
-</robot>
+/home/joshfarina/ros2_ws/src/rbe500_group_project/rrbot_simulation_files/rrbot_description/urdf/rrbot.urdf.xacro

File: install/rrbot_description/share/rrbot_description/urdf/rrbot_description.urdf.xacro (robot description, xacro)
@@ -1,159 +1 @@
-<?xml version="1.0"?>
-<robot xmlns:xacro="http://www.ros.org/wiki/xacro">
-  <xacro:macro name="rrbot" params="parent prefix *origin">
-  <!-- Constants for robot dimensions -->
-  <xacro:property name="mass" value="1" /> <!-- arbitrary value for mass -->
-  <xacro:property name="width" value="0.1" /> <!-- Square dimensions (widthxwidth) of beams -->
-  <xacro:property name="cyl_radius" value="0.3"/><!-- Radius of the revolute joints -->
-  <xacro:property name="cyl_height" value="0.3"/><!--  Height of the revolute joints -->
-  <xacro:property name="l1" value="1" /> <!-- Link 1 --> <!-- arbitrary value for mass -->
-  <xacro:property name="l2" value="1" /> <!-- Link 2 -->
-  <xacro:property name="l3" value="1" /> <!-- Link 3 -->
-  <xacro:property name="l4" value="1" /> <!-- Link 4 -->
-  <xacro:property name="axel_offset" value="0.05" /> <!-- Space btw top of beam and the each joint -->
-  <joint name="${prefix}base_joint" type="fixed">
-    <xacro:insert_block name="origin" />
-    <parent link="${parent}"/>
-    <child link="${prefix}base_link" />
-  </joint>
-  <!-- Base Link -->
-  <link name="${prefix}base_link">
-    <collision>
-      <origin xyz="0 0 ${cyl_height/2}" rpy="0 0 0"/>
-      <geometry>
-        <cylinder length="${cyl_height}" radius = "${cyl_radius}"/>
-      </geometry>
-    </collision>
-    <visual>
-      <origin xyz="0 0 ${cyl_height/2}" rpy="0 0 0"/>
-      <geometry>
-        <cylinder length="${cyl_height}" radius = "${cyl_radius}"/>
-      </geometry>
-      <material name="red"/>
-    </visual>
-    <inertial>
-      <origin xyz="0 0 ${cyl_height/2}" rpy="0 0 0"/>
-      <mass value="${mass}"/>
-      <inertia
-        ixx="${(1/12)*mass*(cyl_height*cyl_height) + 1/4*mass*(cyl_height*cyl_height)}" ixy="0.0" ixz="0.0"
-        iyy="${(1/12)*mass*(cyl_height*cyl_height) + 1/4*mass*(cyl_height*cyl_height)}" iyz="0.0"
-        izz="${(1/2)*mass*cyl_radius*cyl_radius}"/>
-      </inertial>
-    </link>
-    <joint name="joint1" type="continuous">
-        <parent link="base_link"/>
-        <child link="link1"/>
-        <origin xyz="0 0 ${cyl_height}" rpy="0 0 0"/>
-        <axis xyz="0 0 1"/>
-    </joint>
-    <link name="link1">
-        <collision>
-            <origin xyz="0 0 ${l1/2}" rpy="0 0 0"/>
-            <geometry>
-                <box size="${width} ${width} ${l1}"/>
-            </geometry>
-        </collision>
-        <visual>
-            <origin xyz="0 0 ${l1/2}" rpy="0 0 0"/>
-            <geometry>
-                <box size="${width} ${width} ${l1}"/>
-            </geometry>
-            <material name="white"/>
-        </visual>
-        <inertial>
-            <origin xyz="0 0 ${l1/2}" rpy="0 0 0"/>
-            <mass value="${mass}"/>
-            <inertia
-                ixx="${mass / 12.0 * (width*width + l1*l1)}" ixy="0.0" ixz="0.0"
-                iyy="${mass / 12.0 * (width*width + width*width)}" iyz="0.0"
-                izz="${mass / 12.0 * (width*width + l1*l1)}"/>
-        </inertial>
-    </link>
-    <joint name="fixed" type="fixed">
-        <parent link="link1"/>
-        <child link="link2"/>
-        <origin xyz="0 0 ${l1}" rpy="0 0 0"/>
-    </joint>
-    <link name="link2">
-        <collision>
-            <origin xyz="${l2/2} 0 0" rpy="0 0 0"/>
-            <geometry>
-                <box size="${l2} ${width} ${width}"/>
-            </geometry>
-        </collision>
-        <visual>
-            <origin xyz="${l2/2} 0 0" rpy="0 0 0"/>
-           <geometry>
-                <box size="${l2} ${width} ${width}"/>
-           </geometry>
-        </visual>
-        <inertial>
-            <origin xyz="0 0 ${l1/2}" rpy="0 0 0"/>
-            <mass value="${mass}"/>
-            <inertia
-                ixx="${mass / 12.0 * (width*width + width*width)}" ixy="0.0" ixz="0.0"
-                iyy="${mass / 12.0 * (width*width + l1*l1)}" iyz="0.0"
-                izz="${mass / 12.0 * (width*width + l1*l1)}"/>
-        </inertial>
-    </link>
-    <joint name="joint2" type="continuous">
-        <parent link="link2"/>
-        <child link="link3"/>
-        <origin xyz="1 0 0" rpy="0 0 0"/>
-        <axis xyz="0 0 1"/>
-    </joint>
-    <link name="link3">
-        <collision>
-            <origin xyz="${l2/2 + l3} 0 0" rpy="0 0 0"/>
-            <geometry>
-                <box size="${l3} ${width} ${width}"/>
-            </geometry>
-        </collision>
-        <visual>
-            <origin xyz="${l2/2} 0 0" rpy="0 0 0"/>
-           <geometry>
-                <box size="${l3} ${width} ${width}"/>
-           </geometry>
-        </visual>
-        <inertial>
-            <origin xyz="${l2/2} 0 0" rpy="0 0 0"/>
-            <mass value="${mass}"/>
-            <inertia
-                ixx="${mass / 12.0 * (width*width + width*width)}" ixy="0.0" ixz="0.0"
-                iyy="${mass / 12.0 * (width*width + l3*l3)}" iyz="0.0"
-                izz="${mass / 12.0 * (width*width + l3*l3)}"/>
-        </inertial>
-    </link>
-    <link name="link4">
-        <collision>
-            <origin xyz="0 0 ${-l4}" rpy="0 0 0"/>
-            <geometry>
-                <box size="${width} ${width} ${l4}"/>
-            </geometry>
-        </collision>
-        <visual>
-           <origin xyz="${l4} 0 ${-l4}" rpy="0 0 0"/>
-           <geometry>
-                <box size="${width} ${width} ${l4}"/>
-           </geometry>
-           <material name="red"/>
-        </visual>
-        <inertial>
-            <origin xyz="${l2/2 + l3} 0 0" rpy="0 0 0"/>
-            <mass value="${mass}"/>
-            <inertia
-                ixx="${mass / 12.0 * (width*width + width*width)}" ixy="0.0" ixz="0.0"
-                iyy="${mass / 12.0 * (width*width + l4*l4)}" iyz="0.0"
-                izz="${mass / 12.0 * (width*width + l4*l4)}"/>
-        </inertial>
-    </link>
-    <joint name="joint3" type="prismatic">
-        <parent link="link3"/>
-        <child link="link4"/>
-        <origin xyz="0.0 0.0 ${l4/2}" rpy="0 0 0"/>
-        <axis xyz="0 0 1"/>
-        <limit effort="1000.0" lower="0" upper="1.0" velocity="0.5"/>
-        <dynamics damping="0.7"/>
-    </joint>
-  </xacro:macro>
-</robot>
+/home/joshfarina/ros2_ws/src/rbe500_group_project/rrbot_simulation_files/rrbot_description/urdf/rrbot_description.urdf.xacro

File: install/rrbot_description/share/rrbot_description/urdf/rrbot_description_bryan.urdf.xacro (robot description, xacro)
@@ -1,146 +1 @@
-<?xml version="1.0"?>
-<robot xmlns:xacro="http://www.ros.org/wiki/xacro">
-  <xacro:macro name="rrbot" params="parent prefix *origin">
-  <!-- Constants for robot dimensions -->
-  <xacro:property name="mass" value="1" /> <!-- arbitrary value for mass -->
-  <xacro:property name="width" value="0.1" /> <!-- Square dimensions (widthxwidth) of beams -->
-  <xacro:property name="height1" value="1" /> <!-- Link 1 -->
-  <xacro:property name="height2" value="1" /> <!-- Link 2 -->
-  <xacro:property name="height3" value="1" /> <!-- Link 3 -->
-  <xacro:property name="camera_link" value="0.05" /> <!-- Size of square 'camera' box -->
-  <xacro:property name="axel_offset" value="0.05" /> <!-- Space btw top of beam and the each joint -->
-  <joint name="${prefix}base_joint" type="continuous">
-    <xacro:insert_block name="origin" />
-    <origin xyz="0 0 0" rpy="0 0 0"/>
-    <dynamics damping="0.7"/>
-    <axis xyz="0 0 1"/>
-    <parent link="${parent}"/>
-    <child link="${prefix}base_link" />
-  </joint>
-  <!-- Base Link -->
-  <link name="${prefix}base_link">
-    <collision>
-      <origin xyz="0 0 ${height1/2}" rpy="0 0 0"/>
-      <geometry>
-        <box size="${width} ${width} ${height1}"/>
-      </geometry>
-    </collision>
-    <visual>
-      <origin xyz="0 0 ${height1/2}" rpy="0 0 0"/>
-      <geometry>
-        <box size="${width} ${width} ${height1}"/>
-      </geometry>
-      <material name="orange"/>
-    </visual>
-    <inertial>
-      <origin xyz="0 0 ${height1/2}" rpy="0 0 0"/>
-      <mass value="${mass}"/>
-      <inertia
-        ixx="${mass / 12.0 * (width*width + height1*height1)}" ixy="0.0" ixz="0.0"
-        iyy="${mass / 12.0 * (height1*height1 + width*width)}" iyz="0.0"
-        izz="${mass / 12.0 * (width*width + width*width)}"/>
-      </inertial>
-    </link>
-    <joint name="${prefix}joint1" type="fixed">
-      <parent link="${prefix}base_link"/>
-      <child link="${prefix}link1"/>
-      <origin xyz="0 ${width} ${height1 - axel_offset}" rpy="0 1.5708 0"/>
-    </joint>
-    <!-- Middle Link -->
-    <link name="${prefix}link1">
-      <collision>
-        <origin xyz="0 0 ${height2/2 - axel_offset}" rpy="0 0 0"/>
-        <geometry>
-          <box size="${width} ${width} ${height2}"/>
-        </geometry>
-      </collision>
-      <visual>
-        <origin xyz="0 0 ${height2/2 - axel_offset}" rpy="0 0 0"/>
-        <geometry>
-          <box size="${width} ${width} ${height2}"/>
-        </geometry>
-        <material name="yellow"/>
-      </visual>
-      <inertial>
-        <origin xyz="0 0 ${height2/2 - axel_offset}" rpy="0 0 0"/>
-        <mass value="${mass}"/>
-        <inertia
-          ixx="${mass / 12.0 * (width*width + height2*height2)}" ixy="0.0" ixz="0.0"
-          iyy="${mass / 12.0 * (height2*height2 + width*width)}" iyz="0.0"
-          izz="${mass / 12.0 * (width*width + width*width)}"/>
-        </inertial>
-      </link>
-      <joint name="${prefix}joint2" type="continuous">
-        <parent link="${prefix}link1"/>
-        <child link="${prefix}link2"/>
-        <origin xyz="0 ${width} ${height2 - axel_offset*2}" rpy="0 0 0"/>
-        <axis xyz="0 0 1"/>
-        <dynamics damping="0.7"/>
-      </joint>
-      <!-- Top Link -->
-      <link name="${prefix}link2">
-        <collision>
-          <origin xyz="0 0 ${height3/2 - axel_offset}" rpy="0 0 0"/>
-          <geometry>
-            <box size="${width} ${width} ${height3}"/>
-          </geometry>
-        </collision>
-        <visual>
-          <origin xyz="0 0 ${height3/2 - axel_offset}" rpy="0 0 0"/>
-          <geometry>
-            <box size="${width} ${width} ${height3}"/>
-          </geometry>
-          <material name="orange"/>
-        </visual>
-        <inertial>
-          <origin xyz="0 0 ${height3/2 - axel_offset}" rpy="0 0 0"/>
-          <mass value="${mass}"/>
-          <inertia
-            ixx="${mass / 12.0 * (width*width + height3*height3)}" ixy="0.0" ixz="0.0"
-            iyy="${mass / 12.0 * (height3*height3 + width*width)}" iyz="0.0"
-            izz="${mass / 12.0 * (width*width + width*width)}"/>
-          </inertial>
-        </link>
-      <!-- Last Joint -->
-      <joint name="${prefix}joint3" type="prismatic">
-        <parent link="${prefix}link2"/>
-        <child link="${prefix}link3"/>
-        <origin xyz="0 ${width*2} ${height2 - axel_offset*2}" rpy="0 0 0"/>
-        <axis xyz="0 0 1"/>
-        <limit effort="1000.0" lower="0" upper="0.4" velocity="0.5"/>
-        <dynamics damping="0.7"/>
-      </joint>
-      <!-- Last Link -->
-      <link name="${prefix}link3">
-        <collision>
-          <origin xyz="0 0 ${height3/2 - axel_offset}" rpy="0 0 0"/>
-          <geometry>
-            <box size="${width} ${width} ${height3}"/>
-          </geometry>
-        </collision>
-        <visual>
-          <origin xyz="0 0 ${height3/2 - axel_offset}" rpy="0 0 0"/>
-          <geometry>
-            <box size="${width} ${width} ${height3}"/>
-          </geometry>
-          <material name="blue"/>
-        </visual>
-        <inertial>
-          <origin xyz="0 0 ${height3/2 - axel_offset}" rpy="0 0 0"/>
-          <mass value="${mass}"/>
-          <inertia
-            ixx="${mass / 12.0 * (width*width + height3*height3)}" ixy="0.0" ixz="0.0"
-            iyy="${mass / 12.0 * (height3*height3 + width*width)}" iyz="0.0"
-            izz="${mass / 12.0 * (width*width + width*width)}"/>
-          </inertial>
-        </link>
-        <joint name="${prefix}tool_joint" type="fixed">
-          <origin xyz="0 0 1" rpy="0 0 0" />
-          <parent link="${prefix}link2"/>
-          <child link="${prefix}tool_link" />
-        </joint>
-        <!-- Tool Link -->
-        <link name="${prefix}tool_link">
-        </link>
-  </xacro:macro>
-</robot>
+/home/joshfarina/ros2_ws/src/rbe500_group_project/rrbot_simulation_files/rrbot_description/urdf/rrbot_description_bryan.urdf.xacro
